File: hw/sch_pcb/TFRPM01A.kicad_pcb (KiCad board)
At the start: 2 copper layers, 30.5 x 40.1 mm, 25 parts, among them J2 CONN1_2, J3 JUMP_2x1, J4 JUMP_5X2, J5 JUMP_3X2, J6 JUMP2_2x1, J7 JUMP_2x1, M1 HOLE, M2 HOLE, M3 HOLE, M4 HOLE, U1 PCF8583, U2 74AHC1G14GV, Y1 Crystal

Commit message: Edit
Parts:
- removed J3: JUMP_2x1, Mlab_Pin_Headers:Straight_2x01
- removed J4: JUMP_5X2, Mlab_Pin_Headers:Straight_2x05
- removed J5: JUMP_3X2, Mlab_Pin_Headers:Straight_2x03
- removed J6: JUMP2_2x1, Mlab_Pin_Headers:Straight_2x01
- removed J7: JUMP_2x1, Mlab_Pin_Headers:Straight_1x02
- removed Y1: Crystal, Mlab_XTAL:Crystal_HC49-U_Vertical
- added J1: HEADER_1x03, Connector_PinHeader_2.54mm:PinHeader_1x03_P2.54mm_Horizontal, F.Cu at (156.0, 44.2)
- added R10: 100R, Mlab_R:SMD-0603, F.Cu at (150.9, 46.3)
- added R7: -, Mlab_R:SMD-0603, F.Cu at (148.3, 81.0)
- added R8: -, Mlab_R:SMD-0603, F.Cu at (142.0, 41.7)
- added U3: MIC5504-3.3YM5, Package_TO_SOT_SMD:SOT-23-5, F.Cu at (148.3, 36.6)
- C1: value 10pF -> 1uF; footprint Mlab_R:SMD-0805 -> Mlab_R:SMD-0603; moved to F.Cu
- C2: value 10pF -> 10uF; moved to F.Cu
- C3, D1, U2: moved to F.Cu
- C4, R2, R3, R5: footprint Mlab_R:SMD-0805 -> Mlab_R:SMD-0603; moved to F.Cu
- D2: value LED -> LED RED; moved to F.Cu
- J2: value CONN1_2 -> SM04B-GHS-TB; footprint Mlab_Pin_Headers:Straight_2x01 -> Connector_JST:JST_GH_SM04B-GHS-TB_1x04-1MP_P1.25mm_Horizontal
- R1: value - -> 470R; footprint Mlab_R:SMD-0805 -> Mlab_R:SMD-0603; moved to F.Cu
- R4: value R -> 180R; footprint Mlab_R:SMD-0805 -> Mlab_R:SMD-0603; moved to F.Cu
- R6: value - -> 0R; footprint Mlab_R:SMD-0805 -> Mlab_R:SMD-0603; moved to F.Cu
- U1: footprint Mlab_IO:SO-8 -> Mlab_IO:SOT176-1; moved to F.Cu
- moved R6 90.2 mm to (138.2, 41.7), turned to 90 degrees
- moved J2 90.1 mm to (111.5, 29.0), turned to -90 degrees
- moved R1 90.0 mm to (138.2, 44.2), turned to -90 degrees
- moved C1 86.6 mm to (152.1, 36.6), turned to 90 degrees
- moved U2 84.9 mm to (142.0, 48.0)
- moved D1 79.8 mm to (116.6, 29.0)
- moved C2 75.1 mm to (153.4, 48.0)
- moved C3 69.6 mm to (138.2, 36.6), turned to 0 degrees
- moved C4 69.5 mm to (142.0, 36.6), turned to 90 degrees
- moved D2 66.0 mm to (135.0, 60.7), turned to 0 degrees
- moved R4 65.6 mm to (139.4, 60.7)
- moved R3 37.9 mm to (134.4, 78.5), turned to 90 degrees
- moved R5 35.6 mm to (148.3, 78.0), turned to 90 degrees
- moved M4 32.8 mm to (163.6, 122.9)
- moved R2 32.7 mm to (133.1, 79.8)
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Connections:
- C1 pad 1: Net-(C1-Pad1) -> +3V3
- C3 pad 1: VCC -> +5V
- C4 pad 1: VCC -> +5V
- D1 pad 1: VCC -> +5V
- J2 pad 1: Net-(J2-Pad1) -> +5V
- J2 pad 2: VCC -> /SCL
- R1 pad 1: VCC -> Net-(R1-Pad1)
- R2 pad 1: VCC -> +3V3
- R2 pad 2: Net-(J4-Pad7) -> /SCL
- R3 pad 1: VCC -> +3V3
- R3 pad 2: Net-(J4-Pad3) -> /SDA
- R4 pad 1: Net-(J6-Pad2) -> Net-(R4-Pad1)
- R5 pad 1: Net-(J2-Pad1) -> Net-(R5-Pad1)
- R6 pad 1: /COUNT -> +5V
- R6 pad 2: GND -> Net-(R1-Pad1)
- U1 pad 1: Net-(C1-Pad1) -> Net-(R4-Pad1)
- U1 pad 2: Net-(C2-Pad1) -> Net-(U1-Pad2)
- U1 pad 3: Net-(J2-Pad1) -> Net-(R5-Pad1)
- U1 pad 5: Net-(J4-Pad3) -> /SDA
- U1 pad 6: Net-(J4-Pad7) -> /SCL
- U1 pad 8: VCC -> +3V3
- U2 pad 1: (no net) -> /COUNT
- U2 pad 2: /COUNT -> Net-(R4-Pad1)
- U2 pad 3: GND -> (no net)
- U2 pad 4: Net-(J6-Pad2) -> (no net)
- U2 pad 5: VCC -> (no net)
Routing:
- net VCC: track 83.6 -> 0.00 mm, vias 2 -> 0
- net Net-(U1-Pad7): track 24.7 -> 0.00 mm, vias 1 -> 0
- net Net-(C1-Pad1): track 23.6 -> 0.00 mm
- net Net-(C2-Pad1): track 16.1 -> 0.00 mm
- net Net-(J4-Pad3): track 12.8 -> 0.00 mm
- net /COUNT: track 11.2 -> 0.00 mm
- net Net-(J4-Pad7): track 9.96 -> 0.00 mm
- net Net-(J6-Pad2): track 9.05 -> 0.00 mm
- net Net-(J2-Pad1): track 7.46 -> 0.00 mm
- net Net-(D2-Pad2): track 3.81 -> 0.00 mm
- net GND: track 2.54 -> 0.00 mm, vias 3 -> 0
- removed copper zone on B.Cu, net GND
- removed copper zone on F.Cu, net GND
Other:
- board size 30.5 x 40.1 mm -> 53.3 x 31.8 mm

Commit message: Edit
Parts:
- added J3: SM04B-GHS-TB, Connector_JST:JST_GH_SM04B-GHS-TB_1x04-1MP_P1.25mm_Horizontal, F.Cu at (125.5, 36.6)
- moved D1 22.6 mm to (130.6, 46.7)
- moved J2 22.6 mm to (125.5, 46.7)

Commit message: edit
Parts:
- removed M1, M3, M4: HOLE, Mlab_Mechanical:MountingHole_3mm
- added C5: 100nF, Mlab_R:SMD-0603, F.Cu at (140.0, 39.1)
- added C6: 100nF, Mlab_R:SMD-0603, F.Cu at (152.4, 34.5)
- moved R5 46.9 mm to (132.6, 33.8)
- moved R7 45.1 mm to (141.0, 36.6), turned to 180 degrees
- moved U1 42.1 mm to (136.3, 37.8), turned to 180 degrees
- moved Me 39.1 mm to (144.5, 41.7)
- moved R2 34.9 mm to (135.6, 45.0)
- moved R3 33.5 mm to (133.7, 45.0)
- moved D2 27.9 mm to (144.1, 34.3)
- moved R4 26.4 mm to (140.2, 34.3)
- moved U3 16.1 mm to (137.7, 48.6)
- moved C1 15.8 mm to (140.7, 47.5), turned to -90 degrees
- moved U2 15.7 mm to (149.6, 34.3), turned to 90 degrees
- moved C4 14.6 mm to (133.7, 48.6), turned to -90 degrees
- moved C3 13.7 mm to (131.2, 48.3), turned to -90 degrees
- moved R1 12.4 mm to (148.3, 37.1), turned to 0 degrees
- moved R6 9.95 mm to (143.7, 49.9), turned to 0 degrees
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- renumbered M2 to Me
Connections:
- U2 pad 1: /COUNT -> (no net)
- U2 pad 2: Net-(R4-Pad1) -> /COUNT
- U2 pad 3: (no net) -> GND
- U2 pad 4: (no net) -> Net-(R4-Pad1)
- U2 pad 5: (no net) -> +3V3
Routing:
- net /SCL: track 0.00 -> 26.8 mm
- net /SDA: track 0.00 -> 24.5 mm, vias 0 -> 2
- net +5V: track 0.00 -> 14.4 mm
- net +3V3: track 0.00 -> 8.03 mm
Other:
- board size 53.3 x 31.8 mm -> 37.5 x 19 mm
- net class Default: via_dia 0.6 -> 0.8
- net class Vcc: via_dia 0.6 -> 0.8

Commit message: Edit
Parts:
- added G***: LOGO, LOGO, F.Cu at (121.4, 127.0)
- C1, C2, C3, C4, C5, C6, D1, D2, J1, J2, J3, Me, R1, R10, R2, R3, R4, R5, R6, R7, R8, U1, U2, U3: moved to B.Cu
- moved R5 107.0 mm to (120.7, 140.2), turned to -90 degrees
- moved C6 106.8 mm to (136.9, 140.2), turned to 90 degrees
- moved R4 106.0 mm to (128.5, 139.7)
- moved D2 106.0 mm to (132.9, 139.7)
- moved U2 105.9 mm to (139.7, 139.7), turned to -90 degrees
- moved J3 101.5 mm to (113.5, 137.4), turned to 90 degrees
- moved R7 100.3 mm to (128.5, 136.1)
- moved U1 99.0 mm to (124.3, 136.1)
- moved J1 96.5 mm to (138.3, 134.9)
- moved C5 94.3 mm to (127.8, 132.6), turned to -90 degrees
- moved D1 91.5 mm to (118.6, 132.3)
- moved Me 91.5 mm to (132.6, 132.3)
- moved R1 87.6 mm to (136.9, 123.9)
- moved R2 84.9 mm to (123.7, 129.0), turned to -90 degrees
- moved R3 84.9 mm to (121.8, 129.0), turned to -90 degrees
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Routing:
- net +3V3: track 8.03 -> 37.8 mm, vias 0 -> 2
- net +5V: track 14.4 -> 38.6 mm, vias 0 -> 4
- net /COUNT: track 0.00 -> 20.6 mm
- net Net-(R4-Pad1): track 0.00 -> 17.2 mm
- net Net-(R5-Pad1): track 0.00 -> 14.5 mm, vias 0 -> 2
- net Net-(C2-Pad1): track 0.00 -> 11.1 mm
- net Net-(R1-Pad1): track 0.00 -> 7.44 mm
- net GND: track 0.00 -> 3.75 mm, vias 0 -> 46
- net Net-(D2-Pad2): track 0.00 -> 1.54 mm
- added copper zone on B.Cu, net GND
- added copper zone on F.Cu, net GND
Other:
- board size 37.5 x 19 mm -> 37.5 x 19.1 mm
- board text added: "2020"
- board text added: "5V"
- board text added: "I2C"
- board text added: "IN"
- board text added: "TFRPM01A"
- board text added: "ThunderFly.cz"
- board text removed: "#INT"
- board text removed: "0x50.. 0x51_"
- board text removed: "2018"
- board text removed: "Addr"
- board text removed: "CNT"
- board text removed: "CNT EN"
- board text removed: "MAX 5V"
- board text removed: "MLAB.CZ"
- board text removed: "MLAB.CZ 2018"
- board text removed: "POWER"
- board text removed: "RTC03A"
- board text removed: "SCL"
- board text removed: "SDA"
- board text removed: "VCC"

Commit message: Úprava popisků.
Parts:
- moved G*** 0.90 mm to (122.0, 127.6)
Other:
- board text added: "+5V"
- board text added: "2019"
- board text added: "PULSE"
- board text removed: "2020"
- board text removed: "5V"

Commit message: Edit
Other:
- board size 37.5 x 19.1 mm -> 37.5 x 19 mm
