File: hw/sch_pcb/TFRPM01B.kicad_pcb (KiCad board)
At the start: 2 copper layers, 37.5 x 19 mm, 25 parts, among them J1 HEADER_1x03, J2 SM04B-GHS-TB, J3 SM04B-GHS-TB, U1 PCF8583, U2 74AHC1G14GV, U3 MIC5504-3.3YM5

Commit message: Edit PCB
Parts:
- M2: renamed from Me; value HOLE -> M3
- U2: footprint Package_SO:TSOP-5_1.65x3.05mm_P0.95mm -> Package_TO_SOT_SMD:SOT-353_SC-70-5
- moved C5 2.84 mm to (128.3, 129.8), turned to 90 degrees
- moved R5 1.54 mm to (119.1, 139.9)
- moved R4 0.91 mm to (129.3, 139.2), turned to -90 degrees
- moved U1 0.76 mm to (124.3, 135.4)
- moved D1 0.57 mm to (118.1, 132.6), turned to -90 degrees
Routing:
- net +3V3: track 37.8 -> 41.7 mm
- net Net-(R5-Pad1): track 14.5 -> 12.4 mm, vias 2 -> 0
- net +5V: track 38.6 -> 36.5 mm
- net GND: track 3.75 -> 1.67 mm, vias 46 -> 47
- net /SDA: track 24.5 -> 25.6 mm
- net Net-(R4-Pad1): track 17.2 -> 16.3 mm
- net /SCL: track 26.8 -> 27.3 mm

Commit message: Edit PCB
Parts:
- moved R7 1.48 mm to (129.8, 136.9)
Routing:
- net GND: track 1.67 -> 9.14 mm, vias 47 -> 55
- net +3V3: track 41.7 -> 39.4 mm
- net Net-(R5-Pad1): track 12.4 -> 14.0 mm
Other:
- board text added: "2020"
- board text added: "TFRPM01B"
- board text removed: "2019"
- board text removed: "TFRPM01A"
