File: hw/sch_pcb/TFRPM01B.kicad_pcb (KiCad board)
At the start: 2 copper layers, 37.5 x 19 mm, 25 parts, among them J1 HEADER_1x03, J2 SM04B-GHS-TB, J3 SM04B-GHS-TB, M2 M3, U1 PCF8583, U2 74AHC1G14GV, U3 MIC5504-3.3YM5

Commit message: Fix screw position dimensions. Fix mounting screm position in the box.
Other:
- net class Default removed
- net class Vcc removed
