File: hw/sch_pcb/TFRPM01B.kicad_sch (KiCad schematic)
At the start: 24 parts, among them J1 HEADER_1x03, J2 SM04B-GHS-TB, J3 SM04B-GHS-TB, M2 M3, U1 PCF8583, U2 74HC1G14GW, U3 MIC5504-3.3YM5

Commit message: Title block updated to TF version.
Other:
- company: Mlab www.mlab.cz -> ThunderFly s.r.o.
- title: RTC03A -> TFRPM01B
Changed lines of the file:
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@@
 (kicad_sch (version 20201015) (generator eeschema)
-  (page 1 1)
   (paper "A4")
   (title_block
-    (title "RTC03A")
-    (date "%F")
-    (company "Mlab www.mlab.cz")
-    (comment 1 "RTC module with counter mode")
-    (comment 2 "romandvorak@mlab.cz")
-    (comment 4 "Open-source")
+    (title "TFRPM01B")
+    (date "2021-01-23")
+    (company "ThunderFly s.r.o.")
+    (comment 1 "RPM measuring device")
+    (comment 2 "Jacho  <info@thunderfly.cz>")
   )
   (junction (at 27.94 168.91) (diameter 1.016) (color 0 0 0 0))
