File: hw/sch_pcb/TFRPM01C.kicad_sch (KiCad schematic)
At the start: 22 parts, among them J1 HEADER_1x03, J2 SM04B-GHS-TB, J3 SM04B-GHS-TB, M2 M3, U1 PCF8583, U2 74HC1G14GW, U3 MIC5504-3.3YM5

Commit message: Edit, generate images
Other:
- note added: "(Edit JP1 for 0x51)"
Changed lines of the file:
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@@
     (stroke (width 0) (type dash) (color 0 0 0 0))
   )
-  (text "Default set 0x50" (at 90.17 97.79 0)
+  (text "(Edit JP1 for 0x51)" (at 88.9 97.79 0)
     (effects (font (size 1.524 1.524)) (justify left bottom))
   )
-  (text "SET I2C ADRESS" (at 109.22 95.25 180)
+  (text "Default set 0x50" (at 90.17 95.25 0)
+    (effects (font (size 1.524 1.524)) (justify left bottom))
+  )
+  (text "SET I2C ADRESS" (at 109.22 92.71 180)
     (effects (font (size 1.524 1.524)) (justify right bottom))
   )

Commit message: Uprava soucastek ve schema
Parts:
- D1: value ZENER-5.6V -> ZENER-6.2V; UST_ID 5c70984512875079b91f88b2 -> (none)
- R10, R3: UST_ID (none) -> 5c70984612875079b91f899f
- R2: UST_ID (none) -> 5c70984512875079b91f8977
- U2: value 74HC1G14GW -> SN74LVC1G14-Q1; UST_ID 5c70984612875079b91f89e9 -> (none)
- U2: value 74HC1G14GW -> SN74LVC1G14-Q1; UST_ID 5c70984712875079b91f8b5e -> (none)
Changed lines of the file:
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@@
       (effects (font (size 1.27 1.27)) hide)
     )
-    (property "UST_ID" "" (id 5) (at 148.59 57.15 0)
+    (property "UST_ID" "5c70984512875079b91f8977" (id 5) (at 148.59 57.15 0)
       (effects (font (size 1.27 1.27)) hide)
     )
@@
       (effects (font (size 1.27 1.27)) hide)
     )
-    (property "UST_ID" "" (id 5) (at 158.75 105.41 0)
+    (property "UST_ID" "5c70984612875079b91f899f" (id 5) (at 158.75 105.41 0)
       (effects (font (size 1.27 1.27)) hide)
     )
@@
       (effects (font (size 1.27 1.27)) hide)
     )
-    (property "UST_ID" "" (id 5) (at 165.1 105.41 0)
+    (property "UST_ID" "5c70984612875079b91f899f" (id 5) (at 165.1 105.41 0)
       (effects (font (size 1.27 1.27)) hide)
     )
@@
       (effects (font (size 1.27 1.27)) (justify left))
     )
-    (property "Value" "ZENER-5.6V" (id 1) (at 45.1866 176.403 90)
+    (property "Value" "ZENER-6.2V" (id 1) (at 45.187 176.403 90)
       (effects (font (size 1.27 1.27)) (justify left))
     )
@@
       (effects (font (size 1.27 1.27)) hide)
     )
-    (property "UST_ID" "5c70984512875079b91f88b2" (id 5) (at 43.18 175.26 0)
+    (property "UST_ID" "" (id 5) (at 43.18 175.26 0)
       (effects (font (size 1.27 1.27)) hide)
     )
@@
     (in_bom yes) (on_board yes)
     (property "Reference" "U2" (id 0) (at 127 55.4482 0))
-    (property "Value" "74HC1G14GW" (id 1) (at 127 57.7596 0))
+    (property "Value" "SN74LVC1G14-Q1" (id 1) (at 127 57.76 0))
     (property "Footprint" "Package_TO_SOT_SMD:SOT-353_SC-70-5" (id 2) (at 127 63.5 0)
       (effects (font (size 1.27 1.27)) hide)
@@
       (effects (font (size 1.27 1.27)) hide)
     )
-    (property "UST_ID" "5c70984612875079b91f89e9" (id 5) (at 127 63.5 0)
+    (property "UST_ID" "" (id 5) (at 127 63.5 0)
       (effects (font (size 1.27 1.27)) hide)
     )
@@
     (in_bom yes) (on_board yes)
     (property "Reference" "U2" (id 0) (at 46.99 137.16 0))
-    (property "Value" "74HC1G14GW" (id 1) (at 58.42 137.16 90))
+    (property "Value" "SN74LVC1G14-Q1" (id 1) (at 58.42 137.16 90))
     (property "Footprint" "Package_TO_SOT_SMD:SOT-353_SC-70-5" (id 2) (at 53.34 137.16 0)
       (effects (font (size 1.27 1.27)) hide)
@@
       (effects (font (size 1.27 1.27)) hide)
     )
-    (property "UST_ID" "5c70984712875079b91f8b5e" (id 5) (at 53.34 137.16 0)
+    (property "UST_ID" "" (id 5) (at 53.34 137.16 0)
       (effects (font (size 1.27 1.27)) hide)
     )
@@
     )
     (path "/00000000-0000-0000-0000-000059ffcb7d"
-      (reference "D1") (unit 1) (value "ZENER-5.6V") (footprint "Mlab_D:Diode-MiniMELF_Standard")
+      (reference "D1") (unit 1) (value "ZENER-6.2V") (footprint "Mlab_D:Diode-MiniMELF_Standard")
     )
     (path "/00000000-0000-0000-0000-00005b1bc617"
@@
     )
     (path "/00000000-0000-0000-0000-00005b1b4dea"
-      (reference "U2") (unit 1) (value "74HC1G14GW") (footprint "Package_TO_SOT_SMD:SOT-353_SC-70-5")
+      (reference "U2") (unit 1) (value "SN74LVC1G14-Q1") (footprint "Package_TO_SOT_SMD:SOT-353_SC-70-5")
     )
     (path "/00000000-0000-0000-0000-00005ded0588"
-      (reference "U2") (unit 2) (value "74HC1G14GW") (footprint "Package_TO_SOT_SMD:SOT-353_SC-70-5")
+      (reference "U2") (unit 2) (value "SN74LVC1G14-Q1") (footprint "Package_TO_SOT_SMD:SOT-353_SC-70-5")
     )
     (path "/00000000-0000-0000-0000-00005de928cf"

Commit message: Doplnění aktuálních součástek pro osazení.
Parts:
- C1: UST_id 5c70984812875079b91f8bc2 -> (none)
- C2, C3: UST_id 5c70984812875079b91f8bbd -> (none)
- C4, C5, C6: UST_id 5c70984812875079b91f8bf2 -> (none)
- D1: UST_ID (none) -> 604b0326128750769e5b0f93; UST_id 5c70984512875079b91f88b2 -> (none)
- D2: UST_id 5c70984412875079b91f8896 -> (none)
- J2, J3: UST_id 5c86273d1287500b4e0280be -> (none)
- R1: value 470R -> 22k; UST_ID 5c70984512875079b91f8959 -> 5c70984712875079b91f8a87; UST_id 5c70984512875079b91f8959 -> (none)
- R10, R3: UST_id 5c70984512875079b91f8962 -> (none)
- R2: value 100R -> 82R; UST_ID 5c70984512875079b91f8977 -> 5c70984512875079b91f8976; UST_id 5c70984512875079b91f8956 -> (none)
- R4: UST_id 5c70984512875079b91f8957 -> (none)
- U1: UST_id 5c70984712875079b91f8b59 -> (none)
- U2: UST_ID (none) -> 604b05e1128750769e5b106e; UST_id 5c70984612875079b91f89e9 -> (none)
- U2: UST_ID (none) -> 604b05e1128750769e5b106e; UST_id 5c70984712875079b91f8b5e -> (none)
- U3: UST_id 5c7255e81287500b4e112ea2 -> (none)
Changed lines of the file:
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@@
       (effects (font (size 1.27 1.27)) hide)
     )
-    (property "UST_id" "5c70984512875079b91f8957" (id 4) (at 111.76 63.5 0)
+    (property "UST_id" "" (id 4) (at 111.76 63.5 0)
       (effects (font (size 1.27 1.27)) hide)
     )
@@
       (effects (font (size 1.27 1.27)) (justify left))
     )
-    (property "Value" "470R" (id 1) (at 140.208 58.293 0)
+    (property "Value" "22k" (id 1) (at 140.208 58.293 0)
       (effects (font (size 1.27 1.27)) (justify left))
     )
@@
       (effects (font (size 1.27 1.27)) hide)
     )
-    (property "UST_id" "5c70984512875079b91f8959" (id 4) (at 138.43 57.15 0)
-      (effects (font (size 1.27 1.27)) hide)
-    )
-    (property "UST_ID" "5c70984512875079b91f8959" (id 5) (at 138.43 57.15 0)
+    (property "UST_id" "" (id 4) (at 138.43 57.15 0)
+      (effects (font (size 1.27 1.27)) hide)
+    )
+    (property "UST_ID" "5c70984712875079b91f8a87" (id 5) (at 138.43 57.15 0)
       (effects (font (size 1.27 1.27)) hide)
     )
@@
       (effects (font (size 1.27 1.27)) (justify right))
     )
-    (property "Value" "100R" (id 1) (at 150.368 58.293 0)
+    (property "Value" "82R" (id 1) (at 150.368 58.293 0)
       (effects (font (size 1.27 1.27)) (justify right))
     )
@@
       (effects (font (size 1.27 1.27)) hide)
     )
-    (property "UST_id" "5c70984512875079b91f8956" (id 4) (at 148.59 57.15 0)
-      (effects (font (size 1.27 1.27)) hide)
-    )
-    (property "UST_ID" "5c70984512875079b91f8977" (id 5) (at 148.59 57.15 0)
+    (property "UST_id" "" (id 4) (at 148.59 57.15 0)
+      (effects (font (size 1.27 1.27)) hide)
+    )
+    (property "UST_ID" "5c70984512875079b91f8976" (id 5) (at 148.59 57.15 0)
       (effects (font (size 1.27 1.27)) hide)
     )
@@
       (effects (font (size 1.27 1.27)) hide)
     )
-    (property "UST_id" "5c70984512875079b91f8962" (id 4) (at 158.75 105.41 0)
+    (property "UST_id" "" (id 4) (at 158.75 105.41 0)
       (effects (font (size 1.27 1.27)) hide)
     )
@@
       (effects (font (size 1.27 1.27)) hide)
     )
-    (property "UST_id" "5c70984512875079b91f8962" (id 4) (at 165.1 105.41 0)
+    (property "UST_id" "" (id 4) (at 165.1 105.41 0)
       (effects (font (size 1.27 1.27)) hide)
     )
@@
       (effects (font (size 1.524 1.524)))
     )
-    (property "UST_id" "5c70984512875079b91f88b2" (id 4) (at 43.18 175.26 0)
-      (effects (font (size 1.27 1.27)) hide)
-    )
-    (property "UST_ID" "" (id 5) (at 43.18 175.26 0)
+    (property "UST_id" "" (id 4) (at 43.18 175.26 0)
+      (effects (font (size 1.27 1.27)) hide)
+    )
+    (property "UST_ID" "604b0326128750769e5b0f93" (id 5) (at 43.18 175.26 0)
       (effects (font (size 1.27 1.27)) hide)
     )
@@
       (effects (font (size 1.27 1.27)) hide)
     )
-    (property "UST_id" "5c70984412875079b91f8896" (id 4) (at 104.14 63.5 0)
+    (property "UST_id" "" (id 4) (at 104.14 63.5 0)
       (effects (font (size 1.27 1.27)) hide)
     )
@@
       (effects (font (size 1.524 1.524)))
     )
-    (property "UST_id" "5c70984812875079b91f8bf2" (id 4) (at 26.67 137.16 0)
+    (property "UST_id" "" (id 4) (at 26.67 137.16 0)
       (effects (font (size 1.27 1.27)) hide)
     )
@@
       (effects (font (size 1.524 1.524)))
     )
-    (property "UST_id" "5c70984812875079b91f8bbd" (id 4) (at 27.94 175.26 0)
+    (property "UST_id" "" (id 4) (at 27.94 175.26 0)
       (effects (font (size 1.27 1.27)) hide)
     )
@@
       (effects (font (size 1.524 1.524)))
     )
-    (property "UST_id" "5c70984812875079b91f8bf2" (id 4) (at 35.56 137.16 0)
+    (property "UST_id" "" (id 4) (at 35.56 137.16 0)
       (effects (font (size 1.27 1.27)) hide)
     )
@@
       (effects (font (size 1.524 1.524)))
     )
-    (property "UST_id" "5c70984812875079b91f8bf2" (id 4) (at 35.56 175.26 0)
+    (property "UST_id" "" (id 4) (at 35.56 175.26 0)
       (effects (font (size 1.27 1.27)) hide)
     )
@@
       (effects (font (size 1.27 1.27)) hide)
     )
-    (property "UST_id" "5c70984812875079b91f8bc2" (id 4) (at 81.28 175.26 0)
+    (property "UST_id" "" (id 4) (at 81.28 175.26 0)
       (effects (font (size 1.27 1.27)) hide)
     )
@@
       (effects (font (size 1.27 1.27)) hide)
     )
-    (property "UST_id" "5c70984812875079b91f8bbd" (id 4) (at 148.59 71.12 0)
+    (property "UST_id" "" (id 4) (at 148.59 71.12 0)
       (effects (font (size 1.27 1.27)) hide)
     )
@@
       (effects (font (size 1.524 1.524)))
     )
-    (property "UST_id" "5c86273d1287500b4e0280be" (id 4) (at 179.07 114.3 0)
+    (property "UST_id" "" (id 4) (at 179.07 114.3 0)
       (effects (font (size 1.27 1.27)) hide)
     )
@@
       (effects (font (size 1.524 1.524)))
     )
-    (property "UST_id" "5c86273d1287500b4e0280be" (id 4) (at 179.07 143.51 0)
+    (property "UST_id" "" (id 4) (at 179.07 143.51 0)
       (effects (font (size 1.27 1.27)) hide)
     )
@@
       (effects (font (size 1.27 1.27)) hide)
     )
-    (property "UST_id" "5c70984612875079b91f89e9" (id 4) (at 127 63.5 0)
-      (effects (font (size 1.27 1.27)) hide)
-    )
-    (property "UST_ID" "" (id 5) (at 127 63.5 0)
+    (property "UST_id" "" (id 4) (at 127 63.5 0)
+      (effects (font (size 1.27 1.27)) hide)
+    )
+    (property "UST_ID" "604b05e1128750769e5b106e" (id 5) (at 127 63.5 0)
       (effects (font (size 1.27 1.27)) hide)
     )
@@
       (effects (font (size 1.27 1.27)) hide)
     )
-    (property "UST_id" "5c70984712875079b91f8b5e" (id 4) (at 53.34 137.16 0)
-      (effects (font (size 1.27 1.27)) hide)
-    )
-    (property "UST_ID" "" (id 5) (at 53.34 137.16 0)
+    (property "UST_id" "" (id 4) (at 53.34 137.16 0)
+      (effects (font (size 1.27 1.27)) hide)
+    )
+    (property "UST_ID" "604b05e1128750769e5b106e" (id 5) (at 53.34 137.16 0)
       (effects (font (size 1.27 1.27)) hide)
     )
@@
       (effects (font (size 1.27 1.27)) hide)
     )
-    (property "UST_id" "5c7255e81287500b4e112ea2" (id 4) (at 67.31 171.45 0)
+    (property "UST_id" "" (id 4) (at 67.31 171.45 0)
       (effects (font (size 1.27 1.27)) hide)
     )
@@
       (effects (font (size 1.524 1.524)) hide)
     )
-    (property "UST_id" "5c70984712875079b91f8b59" (id 4) (at 133.35 113.03 0)
+    (property "UST_id" "" (id 4) (at 133.35 113.03 0)
       (effects (font (size 1.27 1.27)) hide)
     )
@@
     )
     (path "/00000000-0000-0000-0000-00005b1c4727"
-      (reference "R1") (unit 1) (value "470R") (footprint "Mlab_R:SMD-0805")
+      (reference "R1") (unit 1) (value "22k") (footprint "Mlab_R:SMD-0805")
     )
     (path "/00000000-0000-0000-0000-00005ded9c2d"
-      (reference "R2") (unit 1) (value "100R") (footprint "Mlab_R:SMD-0805")
+      (reference "R2") (unit 1) (value "82R") (footprint "Mlab_R:SMD-0805")
     )
     (path "/00000000-0000-0000-0000-000059ffb143"

Commit message: Edit schema
Parts:
- R4: value 180R -> 62R; UST_ID 5c70984512875079b91f8957 -> 5c70984512875079b91f8974
Changed lines of the file:
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@@
     (in_bom yes) (on_board yes)
     (property "Reference" "R4" (id 0) (at 111.76 58.2422 90))
-    (property "Value" "180R" (id 1) (at 111.76 60.5536 90))
+    (property "Value" "62R" (id 1) (at 111.76 60.554 90))
     (property "Footprint" "Mlab_R:SMD-0603" (id 2) (at 111.76 61.722 90)
       (effects (font (size 1.27 1.27)) hide)
@@
       (effects (font (size 1.27 1.27)) hide)
     )
-    (property "UST_ID" "5c70984512875079b91f8957" (id 5) (at 111.76 63.5 0)
+    (property "UST_ID" "5c70984512875079b91f8974" (id 5) (at 111.76 63.5 0)
       (effects (font (size 1.27 1.27)) hide)
     )
@@
     )
     (path "/00000000-0000-0000-0000-00005b1d2dc1"
-      (reference "R4") (unit 1) (value "180R") (footprint "Mlab_R:SMD-0603")
+      (reference "R4") (unit 1) (value "62R") (footprint "Mlab_R:SMD-0603")
     )
     (path "/00000000-0000-0000-0000-000059ffb1aa"

Commit message: Edit schéma
Parts:
- R4: value 62R -> 51R; UST_ID 5c70984512875079b91f8974 -> 5c70984512875079b91f8953
Changed lines of the file:
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@@
     (in_bom yes) (on_board yes)
     (property "Reference" "R4" (id 0) (at 111.76 58.2422 90))
-    (property "Value" "62R" (id 1) (at 111.76 60.554 90))
+    (property "Value" "51R" (id 1) (at 111.76 60.554 90))
     (property "Footprint" "Mlab_R:SMD-0603" (id 2) (at 111.76 61.722 90)
       (effects (font (size 1.27 1.27)) hide)
@@
       (effects (font (size 1.27 1.27)) hide)
     )
-    (property "UST_ID" "5c70984512875079b91f8974" (id 5) (at 111.76 63.5 0)
+    (property "UST_ID" "5c70984512875079b91f8953" (id 5) (at 111.76 63.5 0)
       (effects (font (size 1.27 1.27)) hide)
     )
@@
     )
     (path "/00000000-0000-0000-0000-00005b1d2dc1"
-      (reference "R4") (unit 1) (value "62R") (footprint "Mlab_R:SMD-0603")
+      (reference "R4") (unit 1) (value "51R") (footprint "Mlab_R:SMD-0603")
     )
     (path "/00000000-0000-0000-0000-000059ffb1aa"
