File: hw/sch_pcb/TFRPM01D.kicad_sch (KiCad schematic)
At the start: 28 parts, among them J1 HEADER_1x03, J2 SM04B-GHS-TB, J3 SM04B-GHS-TB, M2 M3, U1 PCF8583, U2 SN74LVC1G14-Q1, U3 MIC5504-3.3YM5

Commit message: Edit BOM
Parts:
- C2, C3: UST_ID (none) -> 5c70984812875079b91f8bf5
- D3: UST_ID (none) -> 5c70984412875079b91f8895
- R10, R3: UST_ID 5c70984612875079b91f899f -> 5c70984512875079b91f8962
- R5: value R -> 130R; UST_ID 5c70984512875079b91f8953 -> 5cd08b17128750448e4542b1
Changed lines of the file:
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@@
       (effects (font (size 1.27 1.27)) hide)
     )
-    (property "UST_ID" "5c70984612875079b91f899f" (id 5) (at 165.1 105.41 0)
+    (property "UST_ID" "5c70984512875079b91f8962" (id 5) (at 165.1 105.41 0)
       (effects (font (size 1.27 1.27)) hide)
     )
@@
       (effects (font (size 1.27 1.27)) hide)
     )
-    (property "UST_ID" "5c70984612875079b91f899f" (id 5) (at 158.75 105.41 0)
+    (property "UST_ID" "5c70984512875079b91f8962" (id 5) (at 158.75 105.41 0)
       (effects (font (size 1.27 1.27)) hide)
     )
@@
       (effects (font (size 1.27 1.27)) hide)
     )
-    (property "UST_ID" "" (id 5) (at 27.94 175.26 0)
+    (property "UST_ID" "5c70984812875079b91f8bf5" (id 5) (at 27.94 175.26 0)
       (effects (font (size 1.27 1.27)) hide)
     )
@@
       (effects (font (size 1.27 1.27)) hide)
     )
-    (property "UST_ID" "" (id 5) (at 148.59 71.12 0)
+    (property "UST_ID" "5c70984812875079b91f8bf5" (id 5) (at 148.59 71.12 0)
       (effects (font (size 1.27 1.27)) hide)
     )
@@
     (in_bom yes) (on_board yes)
     (property "Reference" "R5" (id 0) (at 67.1322 143.51 90))
-    (property "Value" "R" (id 1) (at 69.444 143.51 90))
+    (property "Value" "130R" (id 1) (at 69.444 143.51 90))
     (property "Footprint" "Resistor_SMD:R_0603_1608Metric" (id 2) (at 70.612 143.51 90)
       (effects (font (size 1.27 1.27)) hide)
@@
       (effects (font (size 1.27 1.27)) hide)
     )
-    (property "UST_ID" "5c70984512875079b91f8953" (id 5) (at 72.39 143.51 0)
+    (property "UST_ID" "5cd08b17128750448e4542b1" (id 5) (at 72.39 143.51 0)
       (effects (font (size 1.27 1.27)) hide)
     )
@@
       (effects (font (size 1.27 1.27)) hide)
     )
-    (property "UST_ID" "" (id 5) (at 72.39 135.89 0)
+    (property "UST_ID" "5c70984412875079b91f8895" (id 5) (at 72.39 135.89 0)
       (effects (font (size 1.27 1.27)) hide)
     )
@@
     )
     (path "/0f0d22b0-c2a7-436a-931c-fa4be6782d48"
-      (reference "R5") (unit 1) (value "R") (footprint "Resistor_SMD:R_0603_1608Metric")
+      (reference "R5") (unit 1) (value "130R") (footprint "Resistor_SMD:R_0603_1608Metric")
     )
     (path "/00000000-0000-0000-0000-000059ffb1aa"
