File: hw/sch_pcb/TFRPM01D.kicad_pcb (KiCad board)
At the start: 2 copper layers, 37.5 x 19 mm, 28 parts, among them J1 HEADER_1x03, J2 SM04B-GHS-TB, J3 SM04B-GHS-TB, M2 M3, U1 PCF8583, U2 SN74LVC1G14-Q1, U3 MIC5504-3.3YM5

Commit message: Edit B.FAB
Parts:
- R5: value R -> 130R
Changed lines of the file:
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@@
       (effects (font (size 0.8 0.8) (thickness 0.1)) (justify mirror))
     )
-    (fp_text value "BZX585-B5V6.115" (at 0 -1.4) (layer "B.Fab")
-      (effects (font (size 1 1) (thickness 0.15)) (justify mirror))
-    )
-    (fp_text user "${REFERENCE}" (at 0 1.3) (layer "B.Fab")
+    (fp_text value "BZX585-B5V6.115" (at 0 -1.4) (layer "B.Fab") hide
+      (effects (font (size 1 1) (thickness 0.15)) (justify mirror))
+    )
+    (fp_text user "${REFERENCE}" (at 0 -1.272904) (layer "B.Fab")
       (effects (font (size 1 1) (thickness 0.15)) (justify mirror))
     )
@@
     (property "Sheetfile" "TFRPM01D.kicad_sch")
     (property "Sheetname" "")
-    (property "UST_ID" "5c70984612875079b91f899f")
+    (property "UST_ID" "5c70984512875079b91f8962")
     (property "UST_id" "")
     (attr smd)
@@
       (effects (font (size 0.8 0.8) (thickness 0.1)) (justify mirror))
     )
-    (fp_text value "10k" (at 0 -1.43) (layer "B.Fab")
+    (fp_text value "10k" (at 0 -1.43) (layer "B.Fab") hide
       (effects (font (size 1 1) (thickness 0.15)) (justify mirror))
     )
@@
     (property "Sheetfile" "TFRPM01D.kicad_sch")
     (property "Sheetname" "")
-    (property "UST_ID" "")
+    (property "UST_ID" "5c70984812875079b91f8bf5")
     (property "UST_id" "")
     (attr smd)
@@
       (effects (font (size 0.8 0.8) (thickness 0.1)) (justify mirror))
     )
-    (fp_text value "100nF" (at 0 -1.43) (layer "B.Fab")
+    (fp_text value "100nF" (at 0 -1.43) (layer "B.Fab") hide
       (effects (font (size 1 1) (thickness 0.15)) (justify mirror))
     )
@@
       (effects (font (size 0.8 0.8) (thickness 0.1)) (justify mirror))
     )
-    (fp_text value "51R" (at 0 -1.43 90) (layer "B.Fab")
+    (fp_text value "51R" (at 0 -1.43 90) (layer "B.Fab") hide
       (effects (font (size 1 1) (thickness 0.15)) (justify mirror))
     )
@@
       (effects (font (size 0.8 0.8) (thickness 0.1)) (justify mirror))
     )
-    (fp_text value "22k" (at 0 -1.65 90) (layer "B.Fab")
+    (fp_text value "22k" (at 0 -1.65 90) (layer "B.Fab") hide
       (effects (font (size 1 1) (thickness 0.15)) (justify mirror))
     )
@@
       (effects (font (size 0.8 0.8) (thickness 0.1)) (justify mirror))
     )
-    (fp_text value "82R" (at 0 -1.65 270) (layer "B.Fab")
+    (fp_text value "82R" (at 0 -1.65 270) (layer "B.Fab") hide
       (effects (font (size 1 1) (thickness 0.15)) (justify mirror))
     )
@@
     (property "Sheetfile" "TFRPM01D.kicad_sch")
     (property "Sheetname" "")
-    (property "UST_ID" "5c70984612875079b91f899f")
+    (property "UST_ID" "5c70984512875079b91f8962")
     (property "UST_id" "")
     (attr smd)
@@
       (effects (font (size 0.8 0.8) (thickness 0.1)) (justify mirror))
     )
-    (fp_text value "10k" (at 0 -1.43) (layer "B.Fab")
+    (fp_text value "10k" (at 0 -1.43) (layer "B.Fab") hide
       (effects (font (size 1 1) (thickness 0.15)) (justify mirror))
     )
@@
       (effects (font (size 0.8 0.8) (thickness 0.1)) (justify mirror))
     )
-    (fp_text value "100nF" (at 0 -1.43 90) (layer "B.Fab")
+    (fp_text value "100nF" (at 0 -1.43 90) (layer "B.Fab") hide
       (effects (font (size 1 1) (thickness 0.15)) (justify mirror))
     )
@@
       (effects (font (size 0.8 0.8) (thickness 0.1)) (justify mirror))
     )
-    (fp_text value "100nF" (at 0 -1.43 90) (layer "B.Fab")
+    (fp_text value "100nF" (at 0 -1.43 90) (layer "B.Fab") hide
       (effects (font (size 1 1) (thickness 0.15)) (justify mirror))
     )
@@
       (effects (font (size 1.524 1.524) (thickness 0.3048)) (justify mirror))
     )
-    (fp_text user "${REFERENCE}" (at -3.575 -4.674 180 unlocked) (layer "B.Fab")
+    (fp_text user "${REFERENCE}" (at 1.376 -0.510904 180 unlocked) (layer "B.Fab")
       (effects (font (size 1 1) (thickness 0.2)) (justify mirror))
     )
@@
       (effects (font (size 0.8 0.8) (thickness 0.1)) (justify mirror))
     )
-    (fp_text value "1uF" (at 0 -1.43 270) (layer "B.Fab")
+    (fp_text value "1uF" (at 0 -1.43 270) (layer "B.Fab") hide
       (effects (font (size 1 1) (thickness 0.15)) (justify mirror))
     )
@@
     (property "Sheetfile" "TFRPM01D.kicad_sch")
     (property "Sheetname" "")
-    (property "UST_ID" "")
+    (property "UST_ID" "5c70984812875079b91f8bf5")
     (property "UST_id" "")
     (attr smd)
@@
       (effects (font (size 0.8 0.8) (thickness 0.1)) (justify mirror))
     )
-    (fp_text value "10uF" (at 0 -1.43 90) (layer "B.Fab")
+    (fp_text value "10uF" (at 0 -1.43 90) (layer "B.Fab") hide
       (effects (font (size 1 1) (thickness 0.15)) (justify mirror))
     )
@@
     (property "Sheetfile" "TFRPM01D.kicad_sch")
     (property "Sheetname" "")
-    (property "UST_ID" "5c70984512875079b91f8953")
+    (property "UST_ID" "5cd08b17128750448e4542b1")
     (property "UST_id" "")
     (attr smd)
@@
       (effects (font (size 0.8 0.8) (thickness 0.1)) (justify mirror))
     )
-    (fp_text value "R" (at 0 -1.43 90) (layer "B.Fab")
+    (fp_text value "130R" (at 0 -1.43 90) (layer "B.Fab") hide
       (effects (font (size 1 1) (thickness 0.15)) (justify mirror))
     )
@@
     (property "Sheetfile" "TFRPM01D.kicad_sch")
     (property "Sheetname" "")
-    (property "UST_ID" "")
-    (property "UST_id" "")
-    (attr smd)
+    (property "UST_ID" "5c70984412875079b91f8895")
+    (property "UST_id" "")
+    (attr smd)
